File: Nivara Controls (KiCad)/Driver_RS485.kicad_sch (KiCad schematic)
At the start: 1 part, among them U3 MAX3485

Commit message: Actualization
Parts:
- removed U3: MAX3485, Package_SO:SOIC-8_3.9x4.9mm_P1.27mm, symbol Interface_UART:MAX3485
- added C29992406: ~, RS485-MODULE:C2992406, symbol PCM_SL_Connectors:C2992406

Commit message: TVS
Parts:
- added C1: C_1206, PCM_Capacitor_SMD_AKL:C_1206_3216Metric, symbol PCM_Capacitor_US_AKL:C_1206
- added D1: SM712, PCM_Package_TO_SOT_SMD_AKL:SOT-23, symbol PCM_Diode_TVS_AKL:SM712
- renumbered C29992406 to C2992406
Connections:
- net +3.3V: now reaches C2992406.1 (VCC)
- net GND: now reaches C2992406.2 (GND)
- net UART_IN: now reaches C2992406.3 (TXD)
- net UART_OUT: now reaches C2992406.4 (RXD)
- net GPIO_control: now reaches C2992406.5 (CON)
- net RS485-B: now reaches C2992406.8 (B)
- net RS485-A: now reaches C2992406.9 (A)
Other:
- note removed: "CONEXION HALF-DUPLEX"
- moved on the sheet: C2992406

Commit message: Actualization
Connections:
- net +3.3V: now also C1.1, D1.2 (A2)
- net GND: now also C1.2, D1.1 (A1), D1.3 (Com)
Other:
- moved on the sheet: D1
