File: Nivara Controls (KiCad)/Driver_RS485.kicad_sch (KiCad schematic)
At the start: 3 parts

Commit message: Actualización
Other:
- moved on the sheet: C1, C2992406, D1

Commit message: Esquemático a PCB (ver errores)
Parts:
- renumbered D1 to D2
Changed lines of the file:
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@@
 		(on_board yes)
 		(dnp no)
-		(fields_autoplaced yes)
-		(property "Reference" "D1"
-			(at 98.4885 66.04 0)
+		(property "Reference" "D2"
+			(at 98.552 66.04 0)
 			(effects
 				(font
@@
 			(project ""
 				(path "/42622735-4343-4315-af64-a45701a752b6/711b914f-41ac-411e-bef3-8ade05c9a19b/0e992bd9-df1d-46c0-8773-93ffa0ff8af8"
-					(reference "D1")
+					(reference "D2")
 					(unit 1)
 				)
