File: Nivara Controls (KiCad)/Placa_Nivara.kicad_sch (KiCad schematic)
At the start: 3 parts, among them U2 ESP32-S3-WROOM-1

Commit message: Actualización
Changed lines of the file:
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@@
 	(hierarchical_label "RLY_1_NC"
 		(shape output)
-		(at 36.83 31.75 0)
+		(at 227.33 157.48 0)
 		(effects
 			(font
@@
 	(hierarchical_label "RLY_1_NO"
 		(shape output)
-		(at 36.83 34.29 0)
+		(at 227.33 160.02 0)
 		(effects
 			(font
@@
 	(hierarchical_label "RLY_2_NC"
 		(shape output)
-		(at 16.51 31.75 0)
+		(at 207.01 157.48 0)
 		(effects
 			(font
@@
 	(hierarchical_label "PNP_input_1"
 		(shape input)
-		(at 58.42 45.72 0)
+		(at 53.34 142.24 0)
 		(effects
 			(font
@@
 	(hierarchical_label "NPN_input_1"
 		(shape input)
-		(at 58.42 26.67 0)
+		(at 53.34 123.19 0)
 		(effects
 			(font
@@
 	(hierarchical_label "NPN_input_2"
 		(shape input)
-		(at 58.42 29.21 0)
+		(at 53.34 125.73 0)
 		(effects
 			(font
@@
 	(hierarchical_label "PNP_OUT_1"
 		(shape output)
-		(at 82.55 45.72 0)
+		(at 77.47 142.24 0)
 		(effects
 			(font
@@
 	(hierarchical_label "PNP_input_2"
 		(shape input)
-		(at 58.42 48.26 0)
+		(at 53.34 144.78 0)
 		(effects
 			(font
@@
 	(hierarchical_label "PNP_OUT_2"
 		(shape output)
-		(at 82.55 48.26 0)
+		(at 77.47 144.78 0)
 		(effects
 			(font
@@
 	(hierarchical_label "NPN_OUT_1"
 		(shape output)
-		(at 82.55 26.67 0)
+		(at 77.47 123.19 0)
 		(effects
 			(font
@@
 	(hierarchical_label "NPN_OUT_2"
 		(shape output)
-		(at 82.55 29.21 0)
+		(at 77.47 125.73 0)
 		(effects
 			(font
@@
 	(hierarchical_label "RLY_2_NO"
 		(shape output)
-		(at 16.51 34.29 0)
+		(at 207.01 160.02 0)
 		(effects
 			(font
@@
 	(hierarchical_label "RLY_2_COM"
 		(shape output)
-		(at 16.51 29.21 0)
+		(at 207.01 154.94 0)
 		(effects
 			(font
@@
 	(hierarchical_label "RLY_1_COM"
 		(shape output)
-		(at 36.83 29.21 0)
+		(at 227.33 154.94 0)
 		(effects
 			(font
@@
 	)
 	(sheet
-		(at 36.83 16.51)
+		(at 227.33 142.24)
 		(size 17.78 10.16)
 		(exclude_from_sim no)
@@
 		)
 		(property "Sheetname" "RLY_MODULE_1"
-			(at 36.83 15.7984 0)
+			(at 227.33 141.5284 0)
 			(effects
 				(font
@@
 		)
 		(property "Sheetfile" "RLY_MODULE_1.kicad_sch"
-			(at 36.83 27.2546 0)
+			(at 227.33 152.9846 0)
 			(effects
 				(font
@@
 	)
 	(sheet
-		(at 58.42 16.51)
+		(at 53.34 113.03)
 		(size 21.59 7.62)
 		(exclude_from_sim no)
@@
 		)
 		(property "Sheetname" "Input_NPN"
-			(at 58.42 15.7984 0)
+			(at 53.34 112.3184 0)
 			(effects
 				(font
@@
 		)
 		(property "Sheetfile" "Input_NPN.kicad_sch"
-			(at 58.42 24.7146 0)
+			(at 53.34 121.2346 0)
 			(effects
 				(font
@@
 	)
 	(sheet
-		(at 82.55 16.51)
+		(at 77.47 113.03)
 		(size 21.59 7.62)
 		(exclude_from_sim no)
@@
 		)
 		(property "Sheetname" "Output_NPN"
-			(at 82.55 15.7984 0)
+			(at 77.47 112.3184 0)
 			(effects
 				(font
@@
 		)
 		(property "Sheetfile" "Output_NPN.kicad_sch"
-			(at 82.55 24.7146 0)
+			(at 77.47 121.2346 0)
 			(effects
 				(font
@@
 	)
 	(sheet
-		(at 82.55 35.56)
+		(at 77.47 132.08)
 		(size 21.59 7.62)
 		(exclude_from_sim no)
@@
 		)
 		(property "Sheetname" "Output_PNP"
-			(at 82.55 34.8484 0)
+			(at 77.47 131.3684 0)
 			(effects
 				(font
@@
 		)
 		(property "Sheetfile" "Output_PNP.kicad_sch"
-			(at 82.55 43.7646 0)
+			(at 77.47 140.2846 0)
 			(effects
 				(font
@@
 	)
 	(sheet
-		(at 105.41 16.51)
+		(at 54.61 54.61)
 		(size 20.32 5.08)
 		(exclude_from_sim no)
@@
 		)
 		(property "Sheetname" "Powersupply"
-			(at 105.41 15.7984 0)
+			(at 54.61 53.8984 0)
 			(effects
 				(font
@@
 		)
 		(property "Sheetfile" "Powersupply.kicad_sch"
-			(at 105.41 22.1746 0)
+			(at 54.61 60.2746 0)
 			(effects
 				(font
@@
 	)
 	(sheet
-		(at 16.51 16.51)
+		(at 207.01 142.24)
 		(size 17.78 10.16)
 		(exclude_from_sim no)
@@
 		)
 		(property "Sheetname" "RLY_MODULE_2"
-			(at 16.51 15.7984 0)
+			(at 207.01 141.5284 0)
 			(effects
 				(font
@@
 		)
 		(property "Sheetfile" "RLY_MODULE_2.kicad_sch"
-			(at 16.51 27.2546 0)
+			(at 207.01 152.9846 0)
 			(effects
 				(font
@@
 	)
 	(sheet
-		(at 58.42 35.56)
+		(at 53.34 132.08)
 		(size 21.59 7.62)
 		(exclude_from_sim no)
@@
 		)
 		(property "Sheetname" "Input_PNP"
-			(at 58.42 34.8484 0)
+			(at 53.34 131.3684 0)
 			(effects
 				(font
@@
 		)
 		(property "Sheetfile" "Input_PNP.kicad_sch"
-			(at 58.42 43.7646 0)
-			(effects
-				(font
+			(at 53.34 140.2846 0)
+			(effects
+				(font

Commit message: Actualization
Changed lines of the file:
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@@
 	(hierarchical_label "RLY_1_NC"
 		(shape output)
-		(at 227.33 157.48 0)
+		(at 233.68 143.51 0)
 		(effects
 			(font
@@
 	(hierarchical_label "RLY_1_NO"
 		(shape output)
-		(at 227.33 160.02 0)
+		(at 233.68 146.05 0)
 		(effects
 			(font
@@
 	(hierarchical_label "RLY_2_NC"
 		(shape output)
-		(at 207.01 157.48 0)
+		(at 210.82 143.51 0)
 		(effects
 			(font
@@
 	(hierarchical_label "RLY_2_NO"
 		(shape output)
-		(at 207.01 160.02 0)
+		(at 210.82 146.05 0)
 		(effects
 			(font
@@
 	(hierarchical_label "RLY_2_COM"
 		(shape output)
-		(at 207.01 154.94 0)
+		(at 210.82 140.97 0)
 		(effects
 			(font
@@
 	(hierarchical_label "RLY_1_COM"
 		(shape output)
-		(at 227.33 154.94 0)
+		(at 233.68 140.97 0)
 		(effects
 			(font
@@
 		(on_board yes)
 		(dnp no)
-		(fields_autoplaced yes)
 		(property "Reference" "#PWR016"
 			(at 154.94 72.39 0)
@@
 		)
 		(property "Value" "+3.3V"
-			(at 154.94 63.5 0)
+			(at 154.94 64.262 0)
 			(effects
 				(font
@@
 	)
 	(sheet
-		(at 227.33 142.24)
+		(at 233.68 128.27)
 		(size 17.78 10.16)
 		(exclude_from_sim no)
@@
 		)
 		(property "Sheetname" "RLY_MODULE_1"
-			(at 227.33 141.5284 0)
+			(at 233.68 127.5584 0)
 			(effects
 				(font
@@
 		)
 		(property "Sheetfile" "RLY_MODULE_1.kicad_sch"
-			(at 227.33 152.9846 0)
+			(at 233.68 139.0146 0)
 			(effects
 				(font
@@
 	)
 	(sheet
-		(at 207.01 142.24)
+		(at 210.82 128.27)
 		(size 17.78 10.16)
 		(exclude_from_sim no)
@@
 		)
 		(property "Sheetname" "RLY_MODULE_2"
-			(at 207.01 141.5284 0)
+			(at 210.82 127.5584 0)
 			(effects
 				(font
@@
 		)
 		(property "Sheetfile" "RLY_MODULE_2.kicad_sch"
-			(at 207.01 152.9846 0)
-			(effects
-				(font
+			(at 210.82 139.0146 0)
+			(effects
+				(font

Commit message: TVS
Other:
- sheet Driver_RS485 ports: added GPIO_control; removed none
Changed lines of the file:
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@@
+	(wire
+		(pts
+			(xy 92.71 80.01) (xy 92.71 81.28)
+		)
+		(stroke
+			(width 0)
+			(type default)
+		)
+	)
+	(wire
+		(pts
+			(xy 85.09 87.63) (xy 85.09 81.28)
+		)
+		(stroke
+			(width 0)
+			(type default)
+		)
+	)
+	(wire
+		(pts
+			(xy 154.94 156.21) (xy 154.94 158.75)
+		)
+		(stroke
+			(width 0)
+			(type default)
+		)
+	)
+	(wire
+		(pts
+			(xy 92.71 81.28) (xy 109.22 81.28)
+		)
+		(stroke
+			(width 0)
+			(type default)
+		)
+	)
+	(wire
+		(pts
+			(xy 200.66 80.01) (xy 207.01 80.01)
+		)
+		(stroke
+			(width 0)
+			(type default)
+		)
+	)
+	(wire
+		(pts
+			(xy 85.09 95.25) (xy 85.09 99.06)
+		)
+		(stroke
+			(width 0)
+			(type default)
+		)
+	)
 	(wire
 		(pts
@@
 	(wire
 		(pts
-			(xy 92.71 80.01) (xy 92.71 81.28)
-		)
-		(stroke
-			(width 0)
-			(type default)
-		)
-	)
-	(wire
-		(pts
-			(xy 85.09 87.63) (xy 85.09 81.28)
-		)
-		(stroke
-			(width 0)
-			(type default)
-		)
-	)
-	(wire
-		(pts
-			(xy 154.94 156.21) (xy 154.94 158.75)
-		)
-		(stroke
-			(width 0)
-			(type default)
-		)
-	)
-	(wire
-		(pts
-			(xy 92.71 81.28) (xy 109.22 81.28)
-		)
-		(stroke
-			(width 0)
-			(type default)
-		)
-	)
-	(wire
-		(pts
-			(xy 85.09 95.25) (xy 85.09 99.06)
-		)
-		(stroke
-			(width 0)
-			(type default)
-		)
-	)
-	(wire
-		(pts
-			(xy 231.14 80.01) (xy 234.95 80.01)
-		)
-		(stroke
-			(width 0)
-			(type default)
-		)
-	)
-	(wire
-		(pts
 			(xy 92.71 71.12) (xy 96.52 71.12)
 		)
@@
 	(wire
 		(pts
-			(xy 231.14 82.55) (xy 234.95 82.55)
+			(xy 236.22 82.55) (xy 240.03 82.55)
 		)
 		(stroke
@@
 	(wire
 		(pts
-			(xy 200.66 80.01) (xy 207.01 80.01)
+			(xy 236.22 80.01) (xy 240.03 80.01)
 		)
 		(stroke
@@
 	(hierarchical_label "RS485-B"
 		(shape bidirectional)
-		(at 234.95 82.55 0)
+		(at 240.03 82.55 0)
 		(effects
 			(font
@@
 	(hierarchical_label "RS485-A"
 		(shape bidirectional)
-		(at 234.95 80.01 0)
+		(at 240.03 80.01 0)
 		(effects
 			(font
@@
 	)
 	(sheet
-		(at 207.01 76.2)
-		(size 24.13 10.16)
+		(at 207.01 77.47)
+		(size 29.21 11.43)
 		(exclude_from_sim no)
 		(in_bom yes)
@@
 		)
 		(property "Sheetname" "Driver_RS485"
-			(at 207.01 75.4884 0)
+			(at 207.01 76.7584 0)
 			(effects
 				(font
@@
 		)
 		(property "Sheetfile" "Driver_RS485.kicad_sch"
-			(at 207.01 86.9446 0)
+			(at 207.01 89.4846 0)
 			(effects
 				(font
@@
 			)
 		)
-		(pin "RS485-A" output
-			(at 231.14 80.01 0)
+		(pin "GPIO_control" output
+			(at 236.22 86.36 0)
 			(effects
 				(font
@@
 			)
 		)
-		(pin "RS485-B" output
-			(at 231.14 82.55 0)
-			(effects
-				(font
+		(pin "RS485-A" bidirectional
+			(at 236.22 80.01 0)
+			(effects
+				(font
+					(size 1.27 1.27)
+				)
+				(justify right)
+			)
+		)
+		(pin "RS485-B" bidirectional
+			(at 236.22 82.55 0)
+			(effects
+				(font

Commit message: Actualización_RLAY
Other:
- removed sheet RLY_MODULE_2
Changed lines of the file:
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@@
 	(hierarchical_label "RLY_2_NC"
 		(shape output)
-		(at 210.82 143.51 0)
+		(at 220.98 132.08 0)
 		(effects
 			(font
@@
 	(hierarchical_label "RLY_2_NO"
 		(shape output)
-		(at 210.82 146.05 0)
+		(at 220.98 134.62 0)
 		(effects
 			(font
@@
 	(hierarchical_label "RLY_2_COM"
 		(shape output)
-		(at 210.82 140.97 0)
+		(at 220.98 129.54 0)
 		(effects
 			(font
@@
 				)
 			)
-		)
-	)
-	(sheet
-		(at 210.82 128.27)
-		(size 17.78 10.16)
-		(exclude_from_sim no)
-		(in_bom yes)
-		(on_board yes)
-		(dnp no)
-		(fields_autoplaced yes)
-		(stroke
-			(width 0.1524)
-			(type solid)
-		)
-		(fill
-			(color 0 0 0 0.0000)
-		)
-		(property "Sheetname" "RLY_MODULE_2"
-			(at 210.82 127.5584 0)
-			(effects
-				(font
-					(size 1.27 1.27)
-					(thickness 0.254)
-					(bold yes)
-				)
-				(justify left bottom)
-			)
-		)
-		(property "Sheetfile" "RLY_MODULE_2.kicad_sch"
-			(at 210.82 139.0146 0)
-			(effects
-				(font
-					(size 1.27 1.27)
-				)
-				(justify left top)
-				(hide yes)
-			)
-		)
-		(instances
-			(project "Nivara Controls"
-				(path "/42622735-4343-4315-af64-a45701a752b6/711b914f-41ac-411e-bef3-8ade05c9a19b"
-					(page "10")
-				)
-			)

Commit message: Actualization
Other:
- sheet RLY_MODULE_1 renamed RLY_MODULE
- sheet Input_NPN ports: added NPN_INPUT, NPN__IN_+, NPN__IN_-; removed none
- sheet Input_PNP ports: added PNP__INPUT_ESP, PNP__IN_+, PNP__IN_-; removed none
- sheet RLY_MODULE ports: added ON_RLY_1, ON_RLY_2, RLAY_1_COM, RLAY_1_NC, RLAY_1_NO, RLAY_2_COM, RLAY_2_NC, RLAY_2_NO; removed none
- moved on the sheet: C4, R1

Commit message: Actualización
Other:
- added sheet 0mA__10mA_module (0mA__10mA_module.kicad_sch)
- added sheet 0v__10v_Module (0v__10v_Module.kicad_sch)
- added sheet 0v__32v__module (0v__32v__module.kicad_sch)
- added sheet 4mA__20mA_module (4mA__20mA_module.kicad_sch)
- added sheet Digit_module (Digit_module.kicad_sch)
- moved on the sheet: C4, R1, U2

Commit message: Actualization
Other:
- added sheet OUT__4__20 (OUT__4__20.kicad_sch)
- sheet 0mA__10mA_module ports: added SCLK, SDA, SEL; removed none
- sheet Input_NPN ports: added NPN-Digit_1, NPN-Digit_2, NPN_in_1, NPN_in_2; removed NPN_INPUT, NPN__IN_+, NPN__IN_-
- sheet Input_PNP ports: added PNP_Digit_1, PNP_Digit_2, PNP_in_1, PNP_in_2; removed PNP__INPUT_ESP, PNP__IN_+, PNP__IN_-

Commit message: Actualizado
Other:
- sheet 0mA__10mA_module ports: added A_Out; removed SEL
- sheet OUT__4__20 ports: added ASLK_4-20, OUT_4-20, SDA_4-20; removed none
