File: Nivara Controls (KiCad)/Output_NPN.kicad_sch (KiCad schematic)
At the start: 0 parts

Commit message: Actualización
Parts:
- added R28, R29: R_0603, PCM_Resistor_SMD_AKL:R_0603_1608Metric, symbol PCM_Resistor_US_AKL:R_0603
- added U8, U9: GAQY211G2S, EastEDA:GAQY211G2s, symbol EDA:GAQY211G2S
Connections:
- new net: R29.2, U9.1
- new net: R28.2, U8.1
- new net GND: U8.2, U8.3, U9.2, U9.3
- new net NPN_Input_1: R29.1
- new net NPN_input_0: R28.1
- new net NPN_output_0: U8.4
- new net NPN_output_1: U9.4
