File: Nivara Controls (KiCad)/Output_PNP.kicad_sch (KiCad schematic)
At the start: 0 parts

Commit message: Actualización
Parts:
- added R30, R31: R_0603, PCM_Resistor_SMD_AKL:R_0603_1608Metric, symbol PCM_Resistor_US_AKL:R_0603
- added U6, U7: GAQY211G2S, EastEDA:GAQY211G2s, symbol EDA:GAQY211G2S
Connections:
- new net: R30.2, U6.1
- new net: R31.2, U7.1
- new net GND: U6.2, U7.2
- new net PNP_Output_0: U6.3
- new net PNP_Output_1: U7.3
- new net PNP_input_0: R30.1
- new net PNP_input_1: R31.1
- new net VCC: U6.4, U7.4
