File: Nivara Controls (KiCad)/0v__10v_Module.kicad_sch (KiCad schematic)
At the start: 4 parts

Commit message: Esquemático a PCB (ver errores)
Parts:
- renumbered D3 to D4
Changed lines of the file:
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@@
 		(on_board yes)
 		(dnp no)
-		(property "Reference" "D3"
+		(property "Reference" "D4"
 			(at 134.874 59.944 0)
 			(effects
@@
 			(project "Nivara Controls"
 				(path "/42622735-4343-4315-af64-a45701a752b6/711b914f-41ac-411e-bef3-8ade05c9a19b/052994b8-ae64-4dbc-9745-12b0d0d230e0"
-					(reference "D3")
+					(reference "D4")
 					(unit 1)
 				)
