File: Nivara Controls (KiCad)/Input_NPN.kicad_sch (KiCad schematic)
At the start: 0 parts

Commit message: Actualization
Parts:
- added D1: DL4007, PCM_Diode_SMD_AKL:D_MELF, symbol PCM_Diode_AKL:DL4007
- added OC1: LTV-357T-B, PCM_Package_SO_AKL:SO-4_4.4x3.9mm_P2.54mm, symbol PCM_Optocoupler_AKL:LTV-357T-B
- added R5, R6: R_0603, PCM_Resistor_SMD_AKL:R_0603_1608Metric, symbol PCM_Resistor_US_AKL:R_0603
Connections:
- new net: D1.1 (K), OC1.1, R5.2
- new net +3.3V: R6.1
- new net GND: OC1.3
- new net NPN_INPUT: OC1.4, R6.2
- new net NPN__IN_+: R5.1
- new net NPN__IN_-: D1.2 (A), OC1.2

Commit message: Actualización
Parts:
- renumbered R5 to R1, R6 to R2
Changed lines of the file:
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@@
 		(on_board yes)
 		(dnp no)
-		(property "Reference" "R5"
-			(at 97.79 68.834 90)
+		(property "Reference" "R1"
+			(at 97.536 67.056 90)
 			(effects
 				(font
@@
 		)
 		(property "Value" "R_0603"
-			(at 97.79 67.31 90)
-			(effects
-				(font
-					(size 1.27 1.27)
-				)
-				(hide yes)
+			(at 97.536 68.834 90)
+			(effects
+				(font
+					(size 1.27 1.27)
+				)
 			)
 		)
@@
 			(project "Nivara Controls"
 				(path "/42622735-4343-4315-af64-a45701a752b6/711b914f-41ac-411e-bef3-8ade05c9a19b/1d56f2ae-86b2-4303-b6cf-39a6bc4c3d5f"
-					(reference "R5")
+					(reference "R1")
 					(unit 1)
 				)
@@
 		(on_board yes)
 		(dnp no)
-		(fields_autoplaced yes)
 		(property "Reference" "OC1"
 			(at 132.08 77.4699 0)
@@
 		)
 		(property "Value" "LTV-357T-B"
-			(at 132.08 80.0099 0)
+			(at 132.08 79.248 0)
 			(effects
 				(font
@@
 		(on_board yes)
 		(dnp no)
-		(property "Reference" "R6"
-			(at 125.73 67.818 0)
+		(property "Reference" "R2"
+			(at 131.064 64.516 0)
 			(effects
 				(font
@@
 		)
 		(property "Value" "R_0603"
-			(at 120.904 67.31 90)
-			(effects
-				(font
-					(size 1.27 1.27)
-				)
-				(hide yes)
+			(at 133.35 66.294 0)
+			(effects
+				(font
+					(size 1.27 1.27)
+				)
 			)
 		)
@@
 			(project "Nivara Controls"
 				(path "/42622735-4343-4315-af64-a45701a752b6/711b914f-41ac-411e-bef3-8ade05c9a19b/1d56f2ae-86b2-4303-b6cf-39a6bc4c3d5f"
-					(reference "R6")
-					(unit 1)
-				)
+					(reference "R2")
+					(unit 1)
+				)

Commit message: Actualization
Parts:
- added D8: DL4007, PCM_Diode_SMD_AKL:D_MELF, symbol PCM_Diode_AKL:DL4007
- added OC5: LTV-357T-B, PCM_Package_SO_AKL:SO-4_4.4x3.9mm_P2.54mm, symbol PCM_Optocoupler_AKL:LTV-357T-B
- added R16, R17: R_0603, PCM_Resistor_SMD_AKL:R_0603_1608Metric, symbol PCM_Resistor_US_AKL:R_0603
Connections:
- net NPN__IN_- is gone; now on net GND: D1.2 (A), OC1.2
- net +3.3V: now also R17.1
- net GND: now also D8.2 (A), OC5.2, OC5.3
- net NPN_INPUT renamed NPN-Digit_input_1
- net NPN__IN_+ renamed NPN_in_1
- new net: D8.1 (K), OC5.1, R16.2
- new net NPN-Digit_input_2: OC5.4, R17.2
- new net NPN_in_2: R16.1

Commit message: Esquemático a PCB (ver errores)
Parts:
- renumbered D1 to D3, R2 to R50, R1 to R51
Changed lines of the file:
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@@
 		(on_board yes)
 		(dnp no)
-		(property "Reference" "D1"
+		(property "Reference" "D3"
 			(at 111.506 81.534 90)
 			(effects
@@
 			(project ""
 				(path "/42622735-4343-4315-af64-a45701a752b6/711b914f-41ac-411e-bef3-8ade05c9a19b/1d56f2ae-86b2-4303-b6cf-39a6bc4c3d5f"
-					(reference "D1")
+					(reference "D3")
 					(unit 1)
 				)
@@
 		(on_board yes)
 		(dnp no)
-		(property "Reference" "R1"
-			(at 97.536 67.056 90)
+		(property "Reference" "R51"
+			(at 97.028 66.802 90)
 			(effects
 				(font
@@
 			(project "Nivara Controls"
 				(path "/42622735-4343-4315-af64-a45701a752b6/711b914f-41ac-411e-bef3-8ade05c9a19b/1d56f2ae-86b2-4303-b6cf-39a6bc4c3d5f"
-					(reference "R1")
+					(reference "R51")
 					(unit 1)
 				)
@@
 		(on_board yes)
 		(dnp no)
-		(property "Reference" "R2"
+		(property "Reference" "R50"
 			(at 131.064 64.516 0)
 			(effects
@@
 			(project "Nivara Controls"
 				(path "/42622735-4343-4315-af64-a45701a752b6/711b914f-41ac-411e-bef3-8ade05c9a19b/1d56f2ae-86b2-4303-b6cf-39a6bc4c3d5f"
-					(reference "R2")
-					(unit 1)
-				)
+					(reference "R50")
+					(unit 1)
+				)

Commit message: Trabajando en PCB
Parts:
- D3, D8: footprint PCM_Diode_SMD_AKL:D_MELF -> Diode_SMD:D_0805_2012Metric_Pad1.15x1.40mm_HandSolder
Changed lines of the file:
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@@
 			)
 		)
-		(property "Footprint" "PCM_Diode_SMD_AKL:D_MELF"
+		(property "Footprint" "Diode_SMD:D_0805_2012Metric_Pad1.15x1.40mm_HandSolder"
 			(at 106.68 78.74 0)
 			(effects
@@
 			)
 		)
-		(property "Footprint" "PCM_Diode_SMD_AKL:D_MELF"
+		(property "Footprint" "Diode_SMD:D_0805_2012Metric_Pad1.15x1.40mm_HandSolder"
 			(at 106.68 128.27 0)
 			(effects
