File: Nivara Controls (KiCad)/Input_PNP.kicad_sch (KiCad schematic)
At the start: 0 parts

Commit message: Actualization
Parts:
- added D2: DL4007, PCM_Diode_SMD_AKL:D_MELF, symbol PCM_Diode_AKL:DL4007
- added OC2: LTV-357T-B, PCM_Package_SO_AKL:SO-4_4.4x3.9mm_P2.54mm, symbol PCM_Optocoupler_AKL:LTV-357T-B
- added R7, R8: R_0603, PCM_Resistor_SMD_AKL:R_0603_1608Metric, symbol PCM_Resistor_US_AKL:R_0603
Connections:
- new net: D2.1 (K), OC2.1, R7.2
- new net +3.3V: OC2.4
- new net GND: R8.2
- new net PNP__INPUT_ESP: OC2.3, R8.1
- new net PNP__IN_+: R7.1
- new net PNP__IN_-: D2.2 (A), OC2.2

Commit message: Actualization
Parts:
- added D9: DL4007, PCM_Diode_SMD_AKL:D_MELF, symbol PCM_Diode_AKL:DL4007
- added OC6: LTV-357T-B, PCM_Package_SO_AKL:SO-4_4.4x3.9mm_P2.54mm, symbol PCM_Optocoupler_AKL:LTV-357T-B
- added R18, R19: R_0603, PCM_Resistor_SMD_AKL:R_0603_1608Metric, symbol PCM_Resistor_US_AKL:R_0603
Connections:
- net PNP__IN_- is gone; now on net GND: D2.2 (A), OC2.2
- net +3.3V: now also OC6.4
- net GND: now also D9.2 (A), OC6.2, R19.2
- net PNP__INPUT_ESP renamed PNP_Digit_1
- net PNP__IN_+ renamed PNP_in_1
- new net: D9.1 (K), OC6.1, R18.2
- new net PNP_Digit_2: OC6.3, R19.1
- new net PNP_in_2: R18.1
Other:
- moved on the sheet: D2, OC2, R7, R8

Commit message: Actualización
Changed lines of the file:
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@@
 	(generator_version "9.0")
 	(paper "A4")
-	(rectangle
-		(start 55.88 29.21)
-		(end 143.51 77.47)
-		(stroke
-			(width 0)
-			(type default)
-		)
-		(fill
-			(type none)
-		)
-	)
-	(rectangle
-		(start 55.88 85.09)
-		(end 143.51 134.62)
-		(stroke
-			(width 0)
-			(type default)
-		)
-		(fill
-			(type none)
-		)
-	)
 	(junction
 		(at 91.44 114.3)

Commit message: Esquemático a PCB (ver errores)
Parts:
- renumbered D2 to D1
Changed lines of the file:
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@@
 		(on_board yes)
 		(dnp no)
-		(property "Reference" "D2"
+		(property "Reference" "D1"
 			(at 96.266 51.054 90)
 			(effects
@@
 			(project "Nivara Controls"
 				(path "/42622735-4343-4315-af64-a45701a752b6/711b914f-41ac-411e-bef3-8ade05c9a19b/d6d4f6f7-bfd3-43e1-a94b-2993a59c2239"
-					(reference "D2")
+					(reference "D1")
 					(unit 1)
 				)

Commit message: Trabajando en PCB
Parts:
- D1, D9: footprint PCM_Diode_SMD_AKL:D_MELF -> Diode_SMD:D_0805_2012Metric_Pad1.15x1.40mm_HandSolder
Changed lines of the file:
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@@
 			)
 		)
-		(property "Footprint" "PCM_Diode_SMD_AKL:D_MELF"
+		(property "Footprint" "Diode_SMD:D_0805_2012Metric_Pad1.15x1.40mm_HandSolder"
 			(at 91.44 105.41 0)
 			(effects
@@
 			)
 		)
-		(property "Footprint" "PCM_Diode_SMD_AKL:D_MELF"
+		(property "Footprint" "Diode_SMD:D_0805_2012Metric_Pad1.15x1.40mm_HandSolder"
 			(at 91.44 48.26 0)
 			(effects
