File: Nivara Controls (KiCad)/Powersupply.kicad_sch (KiCad schematic)
At the start: 6 parts, among them U1 AP63203WU

Commit message: Actualización
Parts:
- removed C1, C5: C_0805, PCM_Capacitor_SMD_AKL:C_0805_2012Metric, symbol PCM_Capacitor_AKL:C_0805
- removed U1: AP63203WU, Package_TO_SOT_SMD:TSOT-23-6, symbol Regulator_Switching:AP63203WU
- added C10, C8, C9: C_0603, PCM_Capacitor_SMD_AKL:C_0603_1608Metric, symbol PCM_Capacitor_US_AKL:C_0603
- added JP1: SolderJumper_2_Open, symbol Jumper:SolderJumper_2_Open
- added R2, R3: R_0603, PCM_Resistor_SMD_AKL:R_0603_1608Metric, symbol PCM_Resistor_US_AKL:R_0603
- added TP1, TP2, TP3, TP4: TestPoint, symbol Connector:TestPoint
- added U4: AP63203WU, Package_TO_SOT_SMD:TSOT-23-6, symbol Regulator_Switching:AP63203WU
- C2: Voltaje (none) -> 50v
- C3: voltaje (none) -> 50v
Connections:
- net +3.3V: now also JP1.2 (B), TP4.1; no longer L1.2
- net GND: now also C10.1, C9.1, R3.2, U4.4 (GND)
- net VCC: now also TP3.1, U4.2 (EN), U4.3 (IN)
- net at L1.1: now also C3.1, U4.5 (SW); no longer C3.2
- new net: C10.2, C8.2, C9.2, JP1.1 (A), L1.2, R2.1, TP1.1
- new net: C8.1, R2.2, R3.1, TP2.1, U4.1 (FB)
- new net: C3.2, U4.6 (BST)

Commit message: Trabajando en PCB
Parts:
- JP1: footprint (none) -> Jumper:SolderJumper-2_P1.3mm_Open_RoundedPad1.0x1.5mm
- TP1, TP2, TP3, TP4: footprint (none) -> TestPoint:TestPoint_Keystone_5015_Micro_Mini
Changed lines of the file:
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@@
+	(wire
+		(pts
+			(xy 173.99 49.53) (xy 173.99 60.96)
+		)
+		(stroke
+			(width 0)
+			(type default)
+		)
+	)
 	(wire
 		(pts
 			(xy 173.99 72.39) (xy 189.23 72.39)
-		)
-		(stroke
-			(width 0)
-			(type default)
-		)
-	)
-	(wire
-		(pts
-			(xy 173.99 58.42) (xy 173.99 60.96)
 		)
 		(stroke
@@
 			)
 		)
-		(property "Footprint" ""
+		(property "Footprint" "TestPoint:TestPoint_Keystone_5015_Micro_Mini"
 			(at 101.6 69.85 0)
 			(effects
@@
 	(symbol
 		(lib_id "power:+3.3V")
-		(at 173.99 58.42 0)
+		(at 173.99 49.53 0)
 		(unit 1)
 		(exclude_from_sim no)
@@
 		(dnp no)
 		(property "Reference" "#PWR020"
-			(at 173.99 62.23 0)
+			(at 173.99 53.34 0)
 			(effects
 				(font
@@
 		)
 		(property "Value" "+3.3V"
-			(at 173.99 54.102 0)
+			(at 173.99 45.212 0)
 			(effects
 				(font
@@
 		)
 		(property "Footprint" ""
-			(at 173.99 58.42 0)
+			(at 173.99 49.53 0)
 			(effects
 				(font
@@
 		)
 		(property "Datasheet" ""
-			(at 173.99 58.42 0)
+			(at 173.99 49.53 0)
 			(effects
 				(font
@@
 		)
 		(property "Description" "Power symbol creates a global label with name \"+3.3V\""
-			(at 173.99 58.42 0)
+			(at 173.99 49.53 0)
 			(effects
 				(font
@@
 			)
 		)
-		(property "Footprint" ""
+		(property "Footprint" "Jumper:SolderJumper-2_P1.3mm_Open_RoundedPad1.0x1.5mm"
 			(at 173.99 64.77 0)
 			(effects
@@
 			)
 		)
-		(property "Footprint" ""
+		(property "Footprint" "TestPoint:TestPoint_Keystone_5015_Micro_Mini"
 			(at 153.67 83.82 0)
 			(effects
@@
 			)
 		)
-		(property "Footprint" ""
+		(property "Footprint" "TestPoint:TestPoint_Keystone_5015_Micro_Mini"
 			(at 184.15 58.42 0)
 			(effects
@@
 			)
 		)
-		(property "Footprint" ""
+		(property "Footprint" "TestPoint:TestPoint_Keystone_5015_Micro_Mini"
 			(at 207.01 66.04 0)
 			(effects
