File: Nivara Controls (KiCad)/RLY_MODULE_1.kicad_sch (KiCad schematic)
At the start: 0 parts

Commit message: Actualización_RLAY
Parts:
- added U1: LK1802, EastEDA:LK1802, symbol EDA:LK1802
Connections:
- new net +3.3V: U1.5 (COM)
- new net GND: U1.2 (E)
- new net ON_RLY_1: U1.3 (1B)
- new net ON_RLY_2: U1.4 (2B)

Commit message: Actualization
Parts:
- added K1, K2: DS1E-S-DC3V, footprints:RELAY_DS1E_PAN, symbol DS1E-S-DC3V:DS1E-S-DC3V
Connections:
- net +3.3V: now also K1.1 (COIL+), K2.1 (COIL+)
- net at U1.1 (1C): now also K1.6 (COIL-)
- net at U1.6 (2C): now also K2.6 (COIL-)
- new net RLAY_1_COM: K1.7 (COM)
- new net RLAY_1_NC: K1.10 (NC)
- new net RLAY_1_NO: K1.12 (NO)
- new net RLAY_2_COM: K2.7 (COM)
- new net RLAY_2_NC: K2.10 (NC)
- new net RLAY_2_NO: K2.12 (NO)
Other:
- moved on the sheet: U1

Commit message: Actualización
Changed lines of the file:
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@@
 	(wire
 		(pts
-			(xy 101.6 85.09) (xy 81.28 85.09)
+			(xy 101.6 85.09) (xy 85.09 85.09)
 		)
 		(stroke
@@
 	(wire
 		(pts
-			(xy 119.38 85.09) (xy 154.94 85.09)
+			(xy 119.38 85.09) (xy 127 85.09)
 		)
 		(stroke
@@
 	(wire
 		(pts
-			(xy 81.28 85.09) (xy 81.28 87.63)
+			(xy 85.09 85.09) (xy 85.09 87.63)
 		)
 		(stroke
@@
 	(wire
 		(pts
-			(xy 154.94 85.09) (xy 154.94 83.82)
+			(xy 127 85.09) (xy 127 82.55)
 		)
 		(stroke
@@
 	(symbol
 		(lib_id "power:GND")
-		(at 81.28 87.63 0)
+		(at 85.09 87.63 0)
 		(unit 1)
 		(exclude_from_sim no)
@@
 		(dnp no)
 		(property "Reference" "#PWR012"
-			(at 81.28 93.98 0)
+			(at 85.09 93.98 0)
 			(effects
 				(font
@@
 		)
 		(property "Value" "GND"
-			(at 81.28 91.44 0)
+			(at 85.09 91.44 0)
 			(effects
 				(font
@@
 		)
 		(property "Footprint" ""
-			(at 81.28 87.63 0)
+			(at 85.09 87.63 0)
 			(effects
 				(font
@@
 		)
 		(property "Datasheet" ""
-			(at 81.28 87.63 0)
+			(at 85.09 87.63 0)
 			(effects
 				(font
@@
 		)
 		(property "Description" "Power symbol creates a global label with name \"GND\" , ground"
-			(at 81.28 87.63 0)
+			(at 85.09 87.63 0)
 			(effects
 				(font
@@
 	(symbol
 		(lib_id "power:+3.3V")
-		(at 154.94 83.82 0)
+		(at 127 82.55 0)
 		(unit 1)
 		(exclude_from_sim no)
@@
 		(fields_autoplaced yes)
 		(property "Reference" "#PWR09"
-			(at 154.94 87.63 0)
+			(at 127 86.36 0)
 			(effects
 				(font
@@
 		)
 		(property "Value" "+3.3V"
-			(at 154.94 78.74 0)
+			(at 127 77.47 0)
 			(effects
 				(font
@@
 		)
 		(property "Footprint" ""
-			(at 154.94 83.82 0)
+			(at 127 82.55 0)
 			(effects
 				(font
@@
 		)
 		(property "Datasheet" ""
-			(at 154.94 83.82 0)
+			(at 127 82.55 0)
 			(effects
 				(font
@@
 		)
 		(property "Description" "Power symbol creates a global label with name \"+3.3V\""
-			(at 154.94 83.82 0)
-			(effects
-				(font
+			(at 127 82.55 0)
+			(effects
+				(font

Commit message: Actualization
Parts:
- removed K1, K2: DS1E-S-DC3V, footprints:RELAY_DS1E_PAN, symbol DS1E-S-DC3V:DS1E-S-DC3V
- added K3, K4: SRA-24VDC-CL, EastEDA:RELAY-TH_SRA-X-CX, symbol EDA:SRA-24VDC-CL
Connections:
- net RLAY_1_COM: now also K3.2
- net RLAY_1_NC: now also K3.5
- net RLAY_1_NO: now also K3.1
- net RLAY_2_COM: now also K4.5
- net RLAY_2_NC: now also K4.2
- net RLAY_2_NO: now also K4.1
- net at U1.1 (1C): now also K3.4
- net at U1.6 (2C): now also K4.4
- new net VCC: K3.3, K4.3

Commit message: Actualización VCC en el COM de los Relay
Connections:
- net +3.3V is gone; now on net VCC: U1.5 (COM)
Changed lines of the file:
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@@
 	(wire
 		(pts
-			(xy 127 85.09) (xy 127 82.55)
+			(xy 127 81.28) (xy 127 85.09)
 		)
 		(stroke
@@
 	)
 	(symbol
+		(lib_id "power:VCC")
+		(at 127 81.28 0)
+		(unit 1)
+		(exclude_from_sim no)
+		(in_bom yes)
+		(on_board yes)
+		(dnp no)
+		(property "Reference" "#PWR063"
+			(at 127 85.09 0)
+			(effects
+				(font
+					(size 1.27 1.27)
+				)
+				(hide yes)
+			)
+		)
+		(property "Value" "VCC"
+			(at 126.746 77.47 0)
+			(effects
+				(font
+					(size 1.27 1.27)
+				)
+			)
+		)
+		(property "Footprint" ""
+			(at 127 81.28 0)
+			(effects
+				(font
+					(size 1.27 1.27)
+				)
+				(hide yes)
+			)
+		)
+		(property "Datasheet" ""
+			(at 127 81.28 0)
+			(effects
+				(font
+					(size 1.27 1.27)
+				)
+				(hide yes)
+			)
+		)
+		(property "Description" "Power symbol creates a global label with name \"VCC\""
+			(at 127 81.28 0)
+			(effects
+				(font
+					(size 1.27 1.27)
+				)
+				(hide yes)
+			)
+		)
+		(pin "1"
+		)
+		(instances
+			(project "Nivara Controls"
+				(path "/42622735-4343-4315-af64-a45701a752b6/711b914f-41ac-411e-bef3-8ade05c9a19b/046ce629-3f56-4f48-b2c7-d6e93ff2fbb5"
+					(reference "#PWR063")
+					(unit 1)
+				)
+			)
+		)
+	)
+	(symbol
 		(lib_id "EDA:SRA-24VDC-CL")
 		(at 86.36 57.15 0)
@@
 					(unit 1)
 				)
-			)
-		)
-	)
-	(symbol
-		(lib_id "power:+3.3V")
-		(at 127 82.55 0)
-		(unit 1)
-		(exclude_from_sim no)
-		(in_bom yes)
-		(on_board yes)
-		(dnp no)
-		(fields_autoplaced yes)
-		(property "Reference" "#PWR09"
-			(at 127 86.36 0)
-			(effects
-				(font
-					(size 1.27 1.27)
-				)
-				(hide yes)
-			)
-		)
-		(property "Value" "+3.3V"
-			(at 127 77.47 0)
-			(effects
-				(font
-					(size 1.27 1.27)
-				)
-			)
-		)
-		(property "Footprint" ""
-			(at 127 82.55 0)
-			(effects
-				(font
-					(size 1.27 1.27)
-				)
-				(hide yes)
-			)
-		)
-		(property "Datasheet" ""
-			(at 127 82.55 0)
-			(effects
-				(font
-					(size 1.27 1.27)
-				)
-				(hide yes)
-			)
-		)
-		(property "Description" "Power symbol creates a global label with name \"+3.3V\""
-			(at 127 82.55 0)
-			(effects
-				(font
-					(size 1.27 1.27)
-				)
-				(hide yes)
-			)
-		)
-		(pin "1"
-		)
-		(instances
-			(project ""
-				(path "/42622735-4343-4315-af64-a45701a752b6/711b914f-41ac-411e-bef3-8ade05c9a19b/046ce629-3f56-4f48-b2c7-d6e93ff2fbb5"
-					(reference "#PWR09")
-					(unit 1)
-				)
