File: Nivara Controls (KiCad)/OUT__4__20.kicad_sch (KiCad schematic)
At the start: 0 parts

Commit message: Actualizado
Parts:
- added C17, C18: C_0603, PCM_Capacitor_SMD_AKL:C_0603_1608Metric, symbol PCM_Capacitor_US_AKL:C_0603
- added R22, R23, R24: R_0603, PCM_Resistor_SMD_AKL:R_0603_1608Metric, symbol PCM_Resistor_US_AKL:R_0603
- added U3: GP8303-TC50-EW, EastEDA:ESOP-10_L4.9-W3.9-P1.00-LS6.1-BL-EP, symbol EDA:GP8303-TC50-EW
Connections:
- new net: C18.1, R24.2, U3.7 (SET)
- new net: C17.2, U3.10 (V5V)
- new net +3.3V: R22.2, R23.2
- new net ASLK_4-20: R23.1, U3.1 (SLCK)
- new net GND: C17.1, C18.2, R24.1, U3.3 (A0), U3.4 (A1), U3.6 (GND), U3.9 (A2)
- new net OUT_4-20: U3.8 (IOUT)
- new net SDA_4-20: R22.1, U3.2 (SDA)
- new net VCC: U3.5 (VCC)

Commit message: Actualizació Orden de componentes
Parts:
- removed R22, R23: R_0603, PCM_Resistor_SMD_AKL:R_0603_1608Metric, symbol PCM_Resistor_US_AKL:R_0603
