File: Nivara Controls (KiCad)/Nivara Controls.kicad_pcb (KiCad board)
At the start: 2 copper layers, 20 parts, among them J1 Screw_Terminal_2_P5.00mm, J10 Screw_Terminal_6_P5.00mm, J2 Screw_Terminal_2_P5.00mm, J3 Screw_Terminal_2_P5.00mm, J4 Screw_Terminal_4_P5.00mm, J5 Screw_Terminal_2_P5.00mm, J6 Screw_Terminal_2_P5.00mm, J7 Screw_Terminal_3_P5.00mm, J8 Screw_Terminal_3_P5.00mm, J9 Screw_Terminal_4_P5.00mm, U1 AP63203WU, U2 ESP32-S3-WROOM-1, U3 MAX3485

Commit message: Actualización
Parts:
- moved J1 81.8 mm to (32.6, 31.6), turned to 0 degrees
- moved J6 58.8 mm to (103.0, 30.5), turned to 0 degrees
- moved J2 57.1 mm to (45.1, 30.5), turned to 0 degrees
- moved J5 35.0 mm to (91.1, 30.3), turned to 0 degrees
- moved J3 33.2 mm to (57.1, 30.5), turned to 0 degrees
- moved J4 9.39 mm to (69.0, 30.4), turned to 0 degrees
- moved J10 7.85 mm to (76.7, 97.7)
- moved J7 7.85 mm to (60.0, 97.7)
- moved J8 7.85 mm to (43.5, 97.6)
- moved J9 7.85 mm to (108.1, 97.7)

Commit message: ACtual
Parts:
- moved U2 52.8 mm to (118.3, 82.4), turned to -90 degrees

Commit message: Acutalizado
Parts:
- added C1: C_1206, PCM_Capacitor_SMD_AKL:C_1206_3216Metric, F.Cu at (203.0, 31.8)
- added C10: C_0603, PCM_Capacitor_SMD_AKL:C_0603_1608Metric, F.Cu at (201.5, 88.8)
- added C11: C_0603, PCM_Capacitor_SMD_AKL:C_0603_1608Metric, F.Cu at (216.3, 50.1)
- added C12: C_0603, PCM_Capacitor_SMD_AKL:C_0603_1608Metric, F.Cu at (227.6, 62.6)
- added C14: C_0603, PCM_Capacitor_SMD_AKL:C_0603_1608Metric, F.Cu at (222.6, 44.7)
- added C15: C_0603, PCM_Capacitor_SMD_AKL:C_0603_1608Metric, F.Cu at (225.7, 72.2)
- added C16: C_0603, PCM_Capacitor_SMD_AKL:C_0603_1608Metric, F.Cu at (225.7, 74.9)
- added C17: C_0603, PCM_Capacitor_SMD_AKL:C_0603_1608Metric, F.Cu at (161.6, 92.2)
- added C18: C_0603, PCM_Capacitor_SMD_AKL:C_0603_1608Metric, F.Cu at (161.6, 95.0)
- added C2: C_1206, PCM_Capacitor_SMD_AKL:C_1206_3216Metric, F.Cu at (210.9, 93.2)
- added C2992406: ~, RS485-MODULE:C2992406, F.Cu at (189.6, 30.8)
- added C3: C_0603, PCM_Capacitor_SMD_AKL:C_0603_1608Metric, F.Cu at (201.5, 80.6)
- added C8: C_0603, PCM_Capacitor_SMD_AKL:C_0603_1608Metric, F.Cu at (201.5, 83.4)
- added C9: C_0603, PCM_Capacitor_SMD_AKL:C_0603_1608Metric, F.Cu at (201.5, 86.1)
- added D1: DL4007, PCM_Diode_SMD_AKL:D_MELF, F.Cu at (169.2, 72.8)
- added D2: SM712, PCM_Package_TO_SOT_SMD_AKL:SOT-23, F.Cu at (202.3, 35.9)
- added D20: MB24F_C7427849, EastEDA:MBF-SMD_L4.7-W3.8-P2.50-LS6.8-BL, F.Cu at (222.4, 60.3)
- added D3: DL4007, PCM_Diode_SMD_AKL:D_MELF, F.Cu at (193.3, 69.3)
- added D4: MB24F_C7427849, EastEDA:MBF-SMD_L4.7-W3.8-P2.50-LS6.8-BL, F.Cu at (211.1, 47.8)
- added D5: DL4007, PCM_Diode_SMD_AKL:D_MELF, F.Cu at (213.3, 69.3)
- added D6: DL4007, PCM_Diode_SMD_AKL:D_MELF, F.Cu at (213.3, 74.6)
- added D7: SMF24A, PCM_Diode_SMD_AKL:D_SOD-123F, F.Cu at (226.4, 68.8)
- added D8: DL4007, PCM_Diode_SMD_AKL:D_MELF, F.Cu at (193.3, 74.6)
- added D9: DL4007, PCM_Diode_SMD_AKL:D_MELF, F.Cu at (169.2, 78.1)
- added J5: Screw_Terminal_4_P5.00mm, TerminalBlock_Phoenix:TerminalBlock_Phoenix_PT-1,5-4-5.0-H_1x04_P5.00mm_Horizontal, F.Cu at (211.6, 35.0)
- added K3: SRA-24VDC-CL, EastEDA:RELAY-TH_SRA-X-CX, F.Cu at (82.3, 84.0)
- added K4: SRA-24VDC-CL, EastEDA:RELAY-TH_SRA-X-CX, F.Cu at (96.3, 83.9)
- added L1: L_Iron, Inductor_SMD:L_Bourns-SRN6028, F.Cu at (207.7, 83.0)
- added OC1: LTV-357T-B, PCM_Package_SO_AKL:SO-4_4.4x3.9mm_P2.54mm, F.Cu at (184.3, 58.7)
- added OC2: LTV-357T-B, PCM_Package_SO_AKL:SO-4_4.4x3.9mm_P2.54mm, F.Cu at (160.2, 62.2)
- added OC3: LTV-357T-B, PCM_Package_SO_AKL:SO-4_4.4x3.9mm_P2.54mm, F.Cu at (204.3, 58.7)
- added OC4: LTV-357T-B, PCM_Package_SO_AKL:SO-4_4.4x3.9mm_P2.54mm, F.Cu at (204.3, 64.4)
- added OC5: LTV-357T-B, PCM_Package_SO_AKL:SO-4_4.4x3.9mm_P2.54mm, F.Cu at (184.3, 64.4)
- added OC6: LTV-357T-B, PCM_Package_SO_AKL:SO-4_4.4x3.9mm_P2.54mm, F.Cu at (160.2, 67.9)
- added R10: R_0603, PCM_Resistor_SMD_AKL:R_0603_1608Metric, F.Cu at (227.4, 57.2)
- added R11: R_0603, PCM_Resistor_SMD_AKL:R_0603_1608Metric, F.Cu at (216.1, 47.4)
- added R12: R_0603, PCM_Resistor_SMD_AKL:R_0603_1608Metric, F.Cu at (227.4, 59.9)
- added R13: R_0603, PCM_Resistor_SMD_AKL:R_0603_1608Metric, F.Cu at (211.3, 65.3)
- added R14: R_0603, PCM_Resistor_SMD_AKL:R_0603_1608Metric, F.Cu at (222.5, 47.4)
- added R15: R_0603, PCM_Resistor_SMD_AKL:R_0603_1608Metric, F.Cu at (221.4, 68.1)
- added R16: R_0603, PCM_Resistor_SMD_AKL:R_0603_1608Metric, F.Cu at (191.3, 57.2)
- added R17: R_0603, PCM_Resistor_SMD_AKL:R_0603_1608Metric, F.Cu at (191.3, 59.9)
- added R18: R_0603, PCM_Resistor_SMD_AKL:R_0603_1608Metric, F.Cu at (167.2, 66.1)
- added R19: R_0603, PCM_Resistor_SMD_AKL:R_0603_1608Metric, F.Cu at (167.2, 68.8)
- added R2: R_0603, PCM_Resistor_SMD_AKL:R_0603_1608Metric, F.Cu at (205.8, 88.2)
- added R20: R_0603, PCM_Resistor_SMD_AKL:R_0603_1608Metric, F.Cu at (221.4, 70.8)
- added R21: R_0603, PCM_Resistor_SMD_AKL:R_0603_1608Metric, F.Cu at (221.4, 73.5)
- added R22: R_0603, PCM_Resistor_SMD_AKL:R_0603_1608Metric, F.Cu at (157.3, 84.1)
- added R23: R_0603, PCM_Resistor_SMD_AKL:R_0603_1608Metric, F.Cu at (157.3, 86.9)
- added R24: R_0603, PCM_Resistor_SMD_AKL:R_0603_1608Metric, F.Cu at (157.3, 89.6)
- added R25: R_0603, PCM_Resistor_SMD_AKL:R_0603_1608Metric, F.Cu at (222.5, 52.1)
- added R28: R_0603, PCM_Resistor_SMD_AKL:R_0603_1608Metric, F.Cu at (218.1, 90.6)
- added R29: R_0603, PCM_Resistor_SMD_AKL:R_0603_1608Metric, F.Cu at (218.1, 93.4)
- added R3: R_0603, PCM_Resistor_SMD_AKL:R_0603_1608Metric, F.Cu at (205.8, 90.9)
- added R30: R_0603, PCM_Resistor_SMD_AKL:R_0603_1608Metric, F.Cu at (181.4, 90.6)
- added R31: R_0603, PCM_Resistor_SMD_AKL:R_0603_1608Metric, F.Cu at (181.4, 93.4)
- added R4: R_0603, PCM_Resistor_SMD_AKL:R_0603_1608Metric, F.Cu at (211.3, 57.2)
- added R5: R_0603, PCM_Resistor_SMD_AKL:R_0603_1608Metric, F.Cu at (211.3, 59.9)
- added R50: R_0603, PCM_Resistor_SMD_AKL:R_0603_1608Metric, F.Cu at (191.3, 62.6)
- added R51: R_0603, PCM_Resistor_SMD_AKL:R_0603_1608Metric, F.Cu at (191.3, 65.3)
- added R6: R_0603, PCM_Resistor_SMD_AKL:R_0603_1608Metric, F.Cu at (211.3, 62.6)
- added R7: R_0603, PCM_Resistor_SMD_AKL:R_0603_1608Metric, F.Cu at (167.2, 60.7)
- added R8: R_0603, PCM_Resistor_SMD_AKL:R_0603_1608Metric, F.Cu at (167.2, 63.4)
- added R9: R_0603, PCM_Resistor_SMD_AKL:R_0603_1608Metric, F.Cu at (216.1, 44.7)
- added U1: LK1802, EastEDA:LK1802, F.Cu at (174.9, 32.2)
- added U3: GP8303-TC50-EW, EastEDA:ESOP-10_L4.9-W3.9-P1.00-LS6.1-BL-EP, F.Cu at (162.5, 86.8)
- added U4: AP63203WU, Package_TO_SOT_SMD:TSOT-23-6, F.Cu at (210.4, 89.2)
- added U6: GAQY211G2S, EastEDA:GAQY211G2s, F.Cu at (182.5, 84.3)
- added U7: GAQY211G2S, EastEDA:GAQY211G2s, F.Cu at (188.5, 84.3)
- added U8: GAQY211G2S, EastEDA:GAQY211G2s, F.Cu at (219.2, 84.3)
- added U9: GAQY211G2S, EastEDA:GAQY211G2s, F.Cu at (225.2, 84.3)
- moved C2 30.2 mm to (43.3, 70.0)
- moved C3 30.2 mm to (42.7, 74.6)
- moved L1 30.2 mm to (50.1, 71.8)
- moved U1 30.2 mm to (50.1, 63.7)
- moved C1 14.7 mm to (100.3, 57.2)
- moved C5 14.7 mm to (100.3, 60.3)
- moved U3 14.7 mm to (93.9, 58.2)
Connections:
- net /Board_NIVARA/Analof_0_10_OUT_1 renamed /Analof_0_10_OUT_1
- U2 pad 10: unconnected-(U2-GPIO17/U1TXD/ADC2_CH6-Pad10) -> /Board_NIVARA/Driver_RS485/UART_IN
- U2 pad 11: unconnected-(U2-GPIO18/U1RXD/ADC2_CH7/CLK_OUT3-Pad11) -> /Board_NIVARA/Driver_RS485/UART_OUT
- U2 pad 12: unconnected-(U2-GPIO8/TOUCH8/ADC1_CH7/SUBSPICS1-Pad12) -> /Board_NIVARA/0mA__10mA_module/SDA
- U2 pad 15: unconnected-(U2-GPIO3/TOUCH3/ADC1_CH2-Pad15) -> /Board_NIVARA/0v__32v__module/D_0v__32v__
- U2 pad 16: unconnected-(U2-GPIO46-Pad16) -> /Board_NIVARA/RLY_MODULE/ON_RLY_1
- U2 pad 17: unconnected-(U2-GPIO9/TOUCH9/ADC1_CH8/FSPIHD/SUBSPIHD-Pad17) -> /Board_NIVARA/0mA__10mA_module/SCLK
- U2 pad 18: unconnected-(U2-GPIO10/TOUCH10/ADC1_CH9/FSPICS0/FSPIIO4/SUBSPICS0-Pad18) -> /Board_NIVARA/NPN-Digit_1
- U2 pad 19: unconnected-(U2-GPIO11/TOUCH11/ADC2_CH0/FSPID/FSPIIO5/SUBSPID-Pad19) -> /Board_NIVARA/NPN-Digit_2
- U2 pad 20: unconnected-(U2-GPIO12/TOUCH12/ADC2_CH1/FSPICLK/FSPIIO6/SUBSPICLK-Pad20) -> /Board_NIVARA/Input_PNP/PNP_Digit_1
- U2 pad 21: unconnected-(U2-GPIO13/TOUCH13/ADC2_CH2/FSPIQ/FSPIIO7/SUBSPIQ-Pad21) -> /Board_NIVARA/Input_PNP/PNP_Digit_2
- U2 pad 23: unconnected-(U2-GPIO21-Pad23) -> /Board_NIVARA/Output_PNP/PNP_input_0
- U2 pad 26: unconnected-(U2-GPIO45-Pad26) -> /Board_NIVARA/RLY_MODULE/ON_RLY_2
- U2 pad 28: unconnected-(U2-SPIIO6/GPIO35/FSPID/SUBSPID-Pad28) -> /Board_NIVARA/RUN/STOP
- U2 pad 31: unconnected-(U2-GPIO38/FSPIWP/SUBSPIWP-Pad31) -> /Board_NIVARA/Output_PNP/PNP_input_1
- U2 pad 36: /Board_NIVARA/Driver_RS485/UART_OUT -> unconnected-(U2-U0RXD/GPIO44/CLK_OUT2-Pad36)
- U2 pad 37: /Board_NIVARA/Driver_RS485/UART_IN -> unconnected-(U2-U0TXD/GPIO43/CLK_OUT1-Pad37)
- U2 pad 38: unconnected-(U2-GPIO2/TOUCH2/ADC1_CH1-Pad38) -> /Board_NIVARA/Output_NPN/NPN_Input_1
- U2 pad 39: unconnected-(U2-GPIO1/TOUCH1/ADC1_CH0-Pad39) -> /Board_NIVARA/Output_NPN/NPN_input_0
- U2 pad 4: unconnected-(U2-GPIO4/TOUCH4/ADC1_CH3-Pad4) -> /Board_NIVARA/0v__10v_Module/D_0v__10v
- U2 pad 5: unconnected-(U2-GPIO5/TOUCH5/ADC1_CH4-Pad5) -> /Board_NIVARA/Analog_4-20_input_1
- U2 pad 6: unconnected-(U2-GPIO6/TOUCH6/ADC1_CH5-Pad6) -> /Board_NIVARA/Digit_module/Digit_input1_--
- U2 pad 7: unconnected-(U2-GPIO7/TOUCH7/ADC1_CH6-Pad7) -> /Board_NIVARA/Digit_module/Digit_input_2--

Commit message: Trabajando en PCB
Parts:
- removed the C1 at (100.3, 57.2)
- removed the C1 at (203.0, 31.8)
- removed the C2 at (43.3, 70.0)
- removed the C3 at (42.7, 74.6)
- removed C5: C_0805, PCM_Capacitor_SMD_AKL:C_0805_2012Metric
- removed the J5 at (91.1, 30.3)
- removed the L1 at (50.1, 71.8)
- removed the U1 at (50.1, 63.7)
- removed the U1 at (174.9, 32.2)
- removed the U3 at (93.9, 58.2)
- added C1: C_1206, PCM_Capacitor_SMD_AKL:C_1206_3216Metric, F.Cu at (253.4, 177.7)
- added JP1: SolderJumper_2_Open, Jumper:SolderJumper-2_P1.3mm_Open_RoundedPad1.0x1.5mm, F.Cu at (37.6, 194.9)
- added TP1: TestPoint, TestPoint:TestPoint_Keystone_5015_Micro_Mini, F.Cu at (33.4, 191.4)
- added TP2: TestPoint, TestPoint:TestPoint_Keystone_5015_Micro_Mini, F.Cu at (33.3, 195.7)
- added TP3: TestPoint, TestPoint:TestPoint_Keystone_5015_Micro_Mini, F.Cu at (33.3, 200.0)
- added TP4: TestPoint, TestPoint:TestPoint_Keystone_5015_Micro_Mini, F.Cu at (33.4, 180.0)
- added U1: LK1802, EastEDA:LK1802, F.Cu at (87.6, 75.6)
- added U5: GP8201S-TC50-EW, EastEDA:GP8303-TC50-EW, F.Cu at (170.9, 188.2)
- D1, D3, D5, D6, D8, D9: footprint PCM_Diode_SMD_AKL:D_MELF -> Diode_SMD:D_0805_2012Metric_Pad1.15x1.40mm_HandSolder
- moved C2 200.7 mm to (41.0, 200.0), turned to -90 degrees
- moved L1 200.0 mm to (35.4, 184.8)
- moved R10 199.2 mm to (85.2, 196.6), turned to -90 degrees
- moved U4 197.6 mm to (41.1, 191.0), turned to 90 degrees
- moved C3 197.3 mm to (37.7, 190.6), turned to 90 degrees
- moved C10 197.2 mm to (37.7, 198.5), turned to 180 degrees
- moved R12 195.6 mm to (83.9, 192.7), turned to 90 degrees
- moved C9 194.1 mm to (41.0, 195.2), turned to 90 degrees
- moved R28 192.4 mm to (58.6, 198.3)
- moved C12 191.9 mm to (86.5, 192.7), turned to -90 degrees
- moved R2 191.9 mm to (37.4, 180.2)
- moved U8 191.4 mm to (62.9, 194.7)
- moved R3 190.9 mm to (40.8, 186.8), turned to 90 degrees
- moved U9 190.6 mm to (62.9, 184.3)
- moved R9 190.0 mm to (102.0, 196.5), turned to 90 degrees
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
Commit message: PCB
Parts:
- moved C1 174.2 mm to (365.1, 44.1)
- moved C16 174.2 mm to (287.8, 52.9)
- moved D2 174.2 mm to (360.0, 45.0)
- moved D20 174.2 mm to (197.2, 52.5)
- moved D9 174.2 mm to (338.9, 47.1)
- moved OC2 174.2 mm to (330.6, 52.5)
- moved R12 174.2 mm to (195.7, 59.1)
- moved R4 174.2 mm to (237.6, 58.1)
- moved R5 174.2 mm to (239.6, 58.1)
- moved R6 174.2 mm to (246.5, 58.3)
- moved TP1 174.2 mm to (145.2, 57.8)
- moved U3 174.2 mm to (260.3, 49.9)
- moved U8 174.2 mm to (174.6, 61.1)
- moved C10 174.2 mm to (149.5, 64.9)
- moved C11 174.2 mm to (214.7, 59.1)
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
Commit message: Actualizació Orden de componentes
Parts:
- added REF**: MountingHole_2.5mm, MountingHole:MountingHole_2.5mm, F.Cu at (34.6, 90.8)
- added REF**: MountingHole_2.5mm, MountingHole:MountingHole_2.5mm, F.Cu at (119.6, 40.8)
- moved U6 337.5 mm to (65.4, 60.4), turned to 90 degrees
- moved C2992406 332.2 mm to (41.5, 78.9), turned to 90 degrees
- moved R30 328.8 mm to (70.7, 63.7), turned to 180 degrees
- moved U7 326.9 mm to (75.8, 60.4), turned to 90 degrees
- moved C1 322.3 mm to (45.5, 85.2), turned to 90 degrees
- moved R31 318.5 mm to (81.1, 63.4), turned to 180 degrees
- moved D2 316.9 mm to (46.4, 90.3), turned to -90 degrees
- moved D9 270.9 mm to (68.2, 38.1)
- moved OC6 270.9 mm to (68.2, 44.0)
- moved R18 270.9 mm to (67.2, 50.3)
- moved R19 270.9 mm to (69.2, 50.2)
- moved D1 269.4 mm to (61.3, 37.9)
- moved OC2 269.4 mm to (61.3, 44.0)
- moved R7 269.4 mm to (60.3, 50.5)
- moved R8 269.4 mm to (62.6, 50.5)
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Other:
- board outline added: 102.2 x 83 mm

Commit message: rutas
Parts:
- removed REF** (x2): MountingHole_2.5mm, MountingHole:MountingHole_2.5mm
- added REF1: MountingHole_2.5mm, MountingHole:MountingHole_2.5mm, F.Cu at (34.7, 90.8)
- added REF2: MountingHole_2.5mm, MountingHole:MountingHole_2.5mm, F.Cu at (119.6, 40.8)
- moved U1 13.5 mm to (74.0, 78.9)
Routing:
- net GND: track 0.00 -> 555.7 mm, vias 0 -> 1
- net +3.3V: track 0.00 -> 258.6 mm, vias 0 -> 6
- net VCC: track 0.00 -> 181.2 mm, vias 0 -> 3
- net /Board_NIVARA/0mA__10mA_module/SCLK: track 0.00 -> 111.0 mm, vias 0 -> 4
- net /Board_NIVARA/0mA__10mA_module/SDA: track 0.00 -> 107.8 mm, vias 0 -> 2
- net /Board_NIVARA/PNP_OUT_1: track 0.00 -> 100.2 mm, vias 0 -> 1
- net /Board_NIVARA/Analog_4-20_input_1: track 0.00 -> 93.8 mm, vias 0 -> 1
- net /Board_NIVARA/PNP_OUT_2: track 0.00 -> 91.8 mm, vias 0 -> 3
- net /Board_NIVARA/0v__10v_Module/D_0v__10v: track 0.00 -> 77.3 mm, vias 0 -> 6
- net /Board_NIVARA/Input_PNP/PNP_Digit_1: track 0.00 -> 74.3 mm, vias 0 -> 2
- net /Board_NIVARA/Input_PNP/PNP_Digit_2: track 0.00 -> 74.3 mm, vias 0 -> 2
- net /Board_NIVARA/RUN/STOP: track 0.00 -> 74.3 mm, vias 0 -> 2
- net /Board_NIVARA/Driver_RS485/UART_IN: track 0.00 -> 72.5 mm, vias 0 -> 2
- net /Board_NIVARA/Driver_RS485/UART_OUT: track 0.00 -> 62.7 mm
- net /Board_NIVARA/0v__32v__module/D_0v__32v__: track 0.00 -> 61.5 mm, vias 0 -> 2
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Other:
- board size 102.2 x 83 mm -> 101.9 x 82.3 mm
